Commit message: Hovering example modified to desired two positions (y and z) | ros::Time begin added and trajectory_pub.publish(trajectory_msg)

File: rotors_description/urdf/bebop2.xacro (robot description, xacro)
@@ -143,5 +143,5 @@
       enable_visual="true">
       <box size="0.001 0.001 0.001" />
-      <origin xyz="0.1 0 0" rpy="0 0 0" />
+      <origin xyz="0.1 0 0" rpy="0 1.5708 0" />
   </xacro:camera_macro>
 </robot>
